File: full_commissioning_shield.sch (EAGLE design)
At the start: 118 parts, among them IC1 LSM303DLHC, IC2 TLV341A, Q1 BSS138, Q2 BSS138, Q3 NMOS BSS138, U1 ARDUINO-MEGAPRO-5V, U10 LM3405XMK, U11 DS1342U+, U13 TPS563200, U14 MIC5365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

Commit message: Fixed some errors
- Fixed a missing net
- Minor polygon fixes
Parts:
- R35: value 680k -> 580k
Connections:
- net LIGHT_PWM: now also U1.45
Changed lines of the file:
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@@
 <part name="R33" library="rcl" deviceset="R-EU_" device="R0805" value="120k"/>
 <part name="R34" library="rcl" deviceset="R-EU_" device="R0805" value="10k"/>
-<part name="R35" library="rcl" deviceset="R-EU_" device="R0805" value="680k"/>
+<part name="R35" library="rcl" deviceset="R-EU_" device="R0805" value="580k"/>
 <part name="C30" library="rcl" deviceset="C-EU" device="C0805" value="22p"/>
 <part name="C31" library="rcl" deviceset="C-EU" device="C0805" value="100n"/>
@@
 </segment>
 </net>
+<net name="LIGHT_PWM" class="0">
+<segment>
+<pinref part="U1" gate="G$1" pin="45"/>
+<wire x1="99.06" y1="60.96" x2="106.68" y2="60.96" width="0.1524" layer="91"/>
+<label x="106.68" y="60.96" size="1.778" layer="95"/>
+</segment>
+</net>
 </nets>
 </sheet>
@@
 </sheet>
 <sheet>
+<description>GPS</description>
 <plain>
 </plain>

Commit message: Fixed footprint
Fixed Arduino Mega footprint and updated gerber files
Parts:
- removed U1: ARDUINO-MEGAPRO-5V, SparkFun-Boards:ARDUINO-MEGAPRO-5V
- added U12: ARDUINO-MEGAFULL, SparkFun-Boards:ARDUINO-MEGAFULL
Connections:
- net +3V3: now also U12.3.3V; no longer U1.3.3V
- net +5V: now also U12.5V@0, U12.5V@1, U12.5V@2; no longer U1.5V@0, U1.5V@1, U1.5V@2
- net 03: now also U12.A0(RX0); no longer U1.A0(RX0)
- net ACTIVITY_ARD: now also U12.49; no longer U1.49
- net AUDIO: now also U12.A6; no longer U1.A6
- net CO: now also U12.A9; no longer U1.A9
- net CONN_ARD: now also U12.51; no longer U1.51
- net D22: now also U12.22; no longer U1.22
- net D24: now also U12.24; no longer U1.24
- net D36: now also U12.36; no longer U1.36
- net D38: now also U12.38; no longer U1.38
- net D40: now also U12.40; no longer U1.40
- net D42: now also U12.42; no longer U1.42
- net D44: now also U12.44; no longer U1.44
- net D46: now also U12.46; no longer U1.46
- net GND: now also U12.GND@0, U12.GND@1, U12.GND@2, U12.GND@3, U12.GND@4; no longer U1.GND@0, U1.GND@1, U1.GND@2, U1.GND@3, U1.GND@4
- net GPS_INT: now also U12.35; no longer U1.35
- net LED1: now also U12.37; no longer U1.37
- net LED2: now also U12.39; no longer U1.39
- net LED3: now also U12.41; no longer U1.41
- net LED4: now also U12.43; no longer U1.43
- net LIGHT_PWM: now also U12.45; no longer U1.45
- net LUX: now also U12.A15; no longer U1.A15
- net MLDPEV_ARD: now also U12.50; no longer U1.50
- net MLDP_ARD: now also U12.52; no longer U1.52
- net N$33: now also U12.25; no longer U1.25
- net NO2: now also U12.A8; no longer U1.A8
- net RX1_ARD: now also U12.19(RX1); no longer U1.19(RX1)
- net RX3_ARD: now also U12.15(RX3); no longer U1.15(RX3)
- net SCL_5V: now also U12.21(SCL); no longer U1.21(SCL)
- net SDA_5V: now also U12.20(SDA); no longer U1.20(SDA)
- net SW1: now also U12.32; no longer U1.32
- net SW2: now also U12.34; no longer U1.34
- net TX1_ARD: now also U12.18(TX1); no longer U1.18(TX1)
- net TX3_ARD: now also U12.14(TX3); no longer U1.14(TX3)
- net WAKEHW_ARD: now also U12.48; no longer U1.48
- net WAKESW_ARD: now also U12.53; no longer U1.53

Commit message: Minor fixes
Power connector + polygons
Parts:
- POWER: device EAGLE-WR-DC_POWER_JACK_CONNECTORS-rev16b:694103303002 -> EAGLE-WR-DC_POWER_JACK_CONNECTORS-rev17a:694108301002
Changed lines of the file:
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@@
 <part name="R18" library="resistor" deviceset="R-EU_" device="R0805" value="330"/>
 <part name="GND25" library="supply1" deviceset="GND" device=""/>
-<part name="POWER" library="EAGLE-WR-DC_POWER_JACK_CONNECTORS-rev16b" deviceset="694103303002" device=""/>
 <part name="U11" library="Maxim_By_element14_Batch_1" deviceset="DS1341U+" device="" value="DS1342U+"/>
 <part name="GND59" library="supply1" deviceset="GND" device=""/>
@@
 <part name="U14" library="mic5365" deviceset="MIC5365" device=""/>
 <part name="U12" library="SparkFun-Boards" deviceset="ARDUINO-MEGA" device="FULL"/>
+<part name="POWER" library="EAGLE-WR-DC_POWER_JACK_CONNECTORS-rev17a" deviceset="694108301002" device=""/>
 </parts>
 <sheets>
@@
 <instance part="GND6" gate="1" x="147.32" y="101.6"/>
 <instance part="GND2" gate="1" x="53.34" y="101.6"/>
-<instance part="POWER" gate="G$1" x="53.34" y="114.3"/>
 <instance part="FRAME2" gate="G$1" x="0" y="0"/>
 <instance part="U13" gate="G$1" x="127" y="109.22"/>
+<instance part="POWER" gate="G$1" x="53.34" y="114.3"/>
 </instances>
 <busses>
@@
 <junction x="86.36" y="114.3"/>
 <wire x1="53.34" y1="114.3" x2="71.12" y2="114.3" width="0.1524" layer="91"/>
+<pinref part="U13" gate="G$1" pin="VIN"/>
 <pinref part="POWER" gate="G$1" pin="1"/>
-<pinref part="U13" gate="G$1" pin="VIN"/>
-</segment>
-</net>
+</segment>
+</net>
